Commit message: Improved cabinet world

File: instruct_to_policy/models/cabinet_0/cabinet_0.urdf (robot description, URDF)
Before this commit: robot cabinet_0, 3 links, 2 joints
Links:
- added link link
Joints:
- added joint joint_2: type fixed, parent link, child link_2, origin xyz=0 0 0 rpy=1.570796326794897 0 -1.570796326794897

File: instruct_to_policy/models/cabinet_0/cabinet_0.urdf.xacro (robot description, xacro)
@@ -7,4 +7,5 @@
     	</inertial>
   	</xacro:macro>
+	<link name="link"/>
 	<link name="link_0">
 		<visual name="cabinet_door_surface-11">
@@ -570,8 +571,8 @@
 		<xacro:default_inertial mass="10"/>
 	</link>
-	<!-- <joint name="joint_2" type="fixed">
+	<joint name="joint_2" type="fixed">
 		<origin rpy="1.570796326794897 0 -1.570796326794897" xyz="0 0 0"/>
 		<child link="link_2"/>
 		<parent link="link"/>
-	</joint> -->
+	</joint>
 </robot>
