Commit message: added gazebo plugin to publish GT 3D bbox

File: instruct_to_policy/robots/panda/panda.urdf.xacro (robot description, xacro)
@@ -9,7 +9,18 @@
   <!-- problem remains: wrong position, FIXME later -->
   <gazebo>
+    <!-- plugin to publish GT world state to moveit planning scene -->
     <plugin filename="libgazebo_ros_moveit_planning_scene.so" name="gazebo_ros_moveit_planning_scene">
       <topicName>/planning_scene</topicName>
-      <updatePeriod>0.5</updatePeriod>
+      <updatePeriod>1.0</updatePeriod>
+    </plugin>
+    <!-- plugin to publish GT 3D bounding boxes to env node -->
+    <plugin filename="libgazebo_ros_bbox_3d_plugin.so " name="gazebo_ros_bbox_3d_plugin">
+      <updatePeriod>1.0</updatePeriod>
+      <links_to_publish>
+        <link>cabinet::drawer0</link>
+        <link>cabinet::drawer1</link>
+        <link>cabinet::drawer2</link>
+        <link>cabinet::drawer3</link>
+      </links_to_publish>
     </plugin>
   </gazebo>

Commit message: updated cabinet model to get GT handle bbox

File: instruct_to_policy/robots/panda/panda.urdf.xacro (robot description, xacro)
@@ -22,4 +22,8 @@
         <link>cabinet::drawer2</link>
         <link>cabinet::drawer3</link>
+        <link>cabinet::handle_0</link>
+        <link>cabinet::handle_1</link>
+        <link>cabinet::handle_2</link>
+        <link>cabinet::handle_3</link>
       </links_to_publish>
     </plugin>

Commit message: improved physics properties

File: instruct_to_policy/robots/panda/panda.urdf.xacro (robot description, xacro)
@@ -6,4 +6,57 @@
                       joint_limits="${xacro.load_yaml('$(find franka_description)/robots/panda/joint_limits.yaml')}">
   </xacro:franka_robot>
+  <!-- overwrite physics parameters for gripper fingers -->
+  <gazebo reference="$(arg arm_id)_leftfinger">
+    <collision>
+      <max_contacts>10</max_contacts>
+      <surface>
+        <contact>
+          <ode>
+            <kp>100000</kp>
+            <kd>5.0</kd>
+            <max_vel>0</max_vel>
+            <min_depth>0.001</min_depth>
+          </ode>
+        </contact>
+        <friction>
+          <ode>
+            <mu>10</mu>
+            <mu2>10</mu2>
+          </ode>
+          <torsional>
+            <coefficient>10.0</coefficient>
+            <use_patch_radius>true</use_patch_radius>
+            <patch_radius>0.1</patch_radius>
+          </torsional>
+        </friction>
+      </surface>
+    </collision>
+  </gazebo>
+  <gazebo reference="$(arg arm_id)_rightfinger">
+    <collision>
+      <max_contacts>10</max_contacts>
+      <surface>
+        <contact>
+          <ode>
+            <kp>100000</kp>
+            <kd>5.0</kd>
+            <max_vel>0</max_vel>
+            <min_depth>0.001</min_depth>
+          </ode>
+        </contact>
+        <friction>
+          <ode>
+            <mu>10</mu>
+            <mu2>10</mu2>
+          </ode>
+          <torsional>
+            <coefficient>10.0</coefficient>
+            <use_patch_radius>true</use_patch_radius>
+            <patch_radius>0.1</patch_radius>
+          </torsional>
+        </friction>
+      </surface>
+    </collision>
+  </gazebo>
   <!-- gazebo plugin to publish models to moveit planning scene -->
   <!-- problem remains: wrong position, FIXME later -->
