Commit message: Run perception pipeline

File: instruct_to_policy/urdf/panda.urdf.xacro (robot description, xacro)
@@ -3,4 +3,6 @@
   <xacro:include filename="$(find franka_description)/robots/common/franka_robot.xacro"/>
   <xacro:arg name="arm_id" default="panda" />
+  <xacro:arg name="use_gt_planning_scene" default="true" />
+  <xacro:arg name="use_gt_bounding_box" default="true" />
   <xacro:franka_robot arm_id="$(arg arm_id)"
                       joint_limits="${xacro.load_yaml('$(find franka_description)/robots/panda/joint_limits.yaml')}">
@@ -60,25 +62,28 @@
   </gazebo>
   <!-- gazebo plugin to publish models to moveit planning scene -->
-  <!-- problem remains: wrong position, FIXME later -->
   <gazebo>
     <!-- plugin to publish GT world state to moveit planning scene -->
-    <plugin filename="libgazebo_ros_moveit_planning_scene.so" name="gazebo_ros_moveit_planning_scene">
-      <topicName>/planning_scene</topicName>
-      <updatePeriod>3.0</updatePeriod>
-    </plugin>
+    <xacro:if value="$(arg use_gt_planning_scene)">
+      <plugin filename="libgazebo_ros_moveit_planning_scene.so" name="gazebo_ros_moveit_planning_scene">
+        <topicName>/planning_scene</topicName>
+        <updatePeriod>3.0</updatePeriod>
+      </plugin>
+    </xacro:if>
     <!-- plugin to publish GT 3D bounding boxes to env node -->
-    <plugin filename="libgazebo_ros_bbox_3d_plugin.so " name="gazebo_ros_bbox_3d_plugin">
-      <updatePeriod>1.0</updatePeriod>
-      <links_to_publish>
-        <link>cabinet::drawer0</link>
-        <link>cabinet::drawer1</link>
-        <link>cabinet::drawer2</link>
-        <link>cabinet::drawer3</link>
-        <link>cabinet::handle_0</link>
-        <link>cabinet::handle_1</link>
-        <link>cabinet::handle_2</link>
-        <link>cabinet::handle_3</link>
-      </links_to_publish>
-    </plugin>
+    <xacro:if value="$(arg use_gt_bounding_box)">
+      <plugin filename="libgazebo_ros_bbox_3d_plugin.so" name="gazebo_ros_bbox_3d_plugin">
+        <updatePeriod>1.0</updatePeriod>
+        <links_to_publish>
+          <link>cabinet::drawer0</link>
+          <link>cabinet::drawer1</link>
+          <link>cabinet::drawer2</link>
+          <link>cabinet::drawer3</link>
+          <link>cabinet::handle_0</link>
+          <link>cabinet::handle_1</link>
+          <link>cabinet::handle_2</link>
+          <link>cabinet::handle_3</link>
+        </links_to_publish>
+      </plugin>
+    </xacro:if>
   </gazebo>
 </robot>

File: instruct_to_policy/urdf/ur5_robotiq85_gripper.urdf.xacro (robot description, xacro)
@@ -1,4 +1,6 @@
 <?xml version="1.0"?>
 <robot name="ur5" xmlns:xacro="http://www.ros.org/wiki/xacro">
+  <xacro:arg name="use_gt_planning_scene" default="true" />
+  <xacro:arg name="use_gt_bounding_box" default="true" />
   <xacro:include filename="$(find ur_description)/urdf/ur5_joint_limited_robot.urdf.xacro" />
   <xacro:include filename="$(find robotiq_description)/urdf/robotiq_85_gripper.urdf.xacro" />
@@ -32,20 +34,29 @@
     </gripper>
   </gazebo>
+  <!-- gazebo plugin to publish models to moveit planning scene -->
   <gazebo>
     <!-- plugin to publish GT world state to moveit planning scene -->
-    <plugin filename="libgazebo_ros_moveit_planning_scene.so" name="gazebo_ros_moveit_planning_scene">
-      <topicName>/planning_scene</topicName>
-      <updatePeriod>3.0</updatePeriod>
-    </plugin>
+    <xacro:if value="$(arg use_gt_planning_scene)">
+      <plugin filename="libgazebo_ros_moveit_planning_scene.so" name="gazebo_ros_moveit_planning_scene">
+        <topicName>/planning_scene</topicName>
+        <updatePeriod>3.0</updatePeriod>
+      </plugin>
+    </xacro:if>
     <!-- plugin to publish GT 3D bounding boxes to env node -->
-    <plugin filename="libgazebo_ros_bbox_3d_plugin.so " name="gazebo_ros_bbox_3d_plugin">
-      <updatePeriod>1.0</updatePeriod>
-      <links_to_publish>
-        <link>cabinet::drawer0</link>
-        <link>cabinet::drawer1</link>
-        <link>cabinet::drawer2</link>
-        <link>cabinet::drawer3</link>
-      </links_to_publish>
-    </plugin>
+    <xacro:if value="$(arg use_gt_bounding_box)">
+      <plugin filename="libgazebo_ros_bbox_3d_plugin.so" name="gazebo_ros_bbox_3d_plugin">
+        <updatePeriod>1.0</updatePeriod>
+        <links_to_publish>
+          <link>cabinet::drawer0</link>
+          <link>cabinet::drawer1</link>
+          <link>cabinet::drawer2</link>
+          <link>cabinet::drawer3</link>
+          <link>cabinet::handle_0</link>
+          <link>cabinet::handle_1</link>
+          <link>cabinet::handle_2</link>
+          <link>cabinet::handle_3</link>
+        </links_to_publish>
+      </plugin>
+    </xacro:if>
   </gazebo>
 </robot>

Commit message: quick fix and rename drawer[0-3] to drawer_[0-3]

File: instruct_to_policy/urdf/panda.urdf.xacro (robot description, xacro)
@@ -75,8 +75,8 @@
       <plugin filename="libgazebo_ros_bbox_3d_plugin.so" name="gazebo_ros_bbox_3d_plugin">
         <links_to_publish>
-          <link>cabinet::drawer0</link>
-          <link>cabinet::drawer1</link>
-          <link>cabinet::drawer2</link>
-          <link>cabinet::drawer3</link>
+          <link>cabinet::drawer_0</link>
+          <link>cabinet::drawer_1</link>
+          <link>cabinet::drawer_2</link>
+          <link>cabinet::drawer_3</link>
           <link>cabinet::handle_0</link>
           <link>cabinet::handle_1</link>

File: instruct_to_policy/urdf/quadruple_d435_cameras.urdf.xacro (robot description, xacro)
@@ -34,8 +34,8 @@
       <updatePeriod>1.0</updatePeriod>
       <links_to_publish>
-        <link>cabinet::drawer0</link>
-        <link>cabinet::drawer1</link>
-        <link>cabinet::drawer2</link>
-        <link>cabinet::drawer3</link>
+        <link>cabinet::drawer_0</link>
+        <link>cabinet::drawer_1</link>
+        <link>cabinet::drawer_2</link>
+        <link>cabinet::drawer_3</link>
       </links_to_publish>
     </plugin>

File: instruct_to_policy/urdf/triple_d435_cameras.urdf.xacro (robot description, xacro)
@@ -30,8 +30,8 @@
       <updatePeriod>1.0</updatePeriod>
       <links_to_publish>
-        <link>cabinet::drawer0</link>
-        <link>cabinet::drawer1</link>
-        <link>cabinet::drawer2</link>
-        <link>cabinet::drawer3</link>
+        <link>cabinet::drawer_0</link>
+        <link>cabinet::drawer_1</link>
+        <link>cabinet::drawer_2</link>
+        <link>cabinet::drawer_3</link>
       </links_to_publish>
     </plugin>

File: instruct_to_policy/urdf/ur5_robotiq85_gripper.urdf.xacro (robot description, xacro)
@@ -49,8 +49,8 @@
         <updatePeriod>1.0</updatePeriod>
         <links_to_publish>
-          <link>cabinet::drawer0</link>
-          <link>cabinet::drawer1</link>
-          <link>cabinet::drawer2</link>
-          <link>cabinet::drawer3</link>
+          <link>cabinet::drawer_0</link>
+          <link>cabinet::drawer_1</link>
+          <link>cabinet::drawer_2</link>
+          <link>cabinet::drawer_3</link>
           <link>cabinet::handle_0</link>
           <link>cabinet::handle_1</link>
